Commit message: Joint limits were wrong for our robot

File: urdf/rx60l_macro.xacro (robot description, xacro)
@@ -178,5 +178,5 @@
 			<child link="${prefix}staubli_rx60l_link6"/>
 			<axis xyz="0 1 0"/>
-			<limit effort="100" velocity="5.585053606" lower="-1.911135531" upper="2.103121749"/>
+			<limit effort="100" velocity="5.585053606" lower="-1.78" upper="1.86"/>
 		</joint>
 		<joint name="${prefix}joint_6" type="revolute">
@@ -185,5 +185,5 @@
 			<child link="${prefix}staubli_rx60l_link7"/>
 			<axis xyz="0 0 1"/>
-			<limit effort="100" velocity="12.217304764" lower="-4.71238898" upper="4.71238898"/>
+			<limit effort="100" velocity="12.217304764" lower="-6.2" upper="6.2"/>
 		</joint>
 		<joint name="${prefix}joint_6-tool0" type="fixed">

Commit message: changed name to follow package naming convention

File: urdf/rx60l_macro.xacro (robot description, xacro)
@@ -7,5 +7,5 @@
 				<origin xyz="0 0 0" rpy="0 0 0"/>
 				<geometry>
-					<mesh filename="package://staubli/meshes/rx60l/visual/rx60bl_hb.dae" scale="0.001 0.001 0.001"/>
+					<mesh filename="package://staubli_description/meshes/rx60l/visual/rx60bl_hb.dae" scale="0.001 0.001 0.001"/>
 				</geometry>
 				<material name="Yellow">
@@ -16,5 +16,5 @@
 				<origin xyz="0 0 0" rpy="0 0 0"/>
 				<geometry>
-					<mesh filename="package://staubli/meshes/rx60l/collision/rx60bl_hb.stl" scale="0.001 0.001 0.001"/>
+					<mesh filename="package://staubli_description/meshes/rx60l/collision/rx60bl_hb.stl" scale="0.001 0.001 0.001"/>
 				</geometry>
 				<material name="Blue">
@@ -27,5 +27,5 @@
 				<origin xyz="0 0 0" rpy="0 0 0"/>
 				<geometry>
-					<mesh filename="package://staubli/meshes/rx60l/visual/rx60bl_hb1.dae" scale="0.001 0.001 0.001"/>
+					<mesh filename="package://staubli_description/meshes/rx60l/visual/rx60bl_hb1.dae" scale="0.001 0.001 0.001"/>
 				</geometry>
 				<material name="Yellow">
@@ -36,5 +36,5 @@
 				<origin xyz="0 0 0" rpy="0 0 0"/>
 				<geometry>
-					<mesh filename="package://staubli/meshes/rx60l/visual/rx60bl_hb1.dae" scale="0.001 0.001 0.001"/>
+					<mesh filename="package://staubli_description/meshes/rx60l/visual/rx60bl_hb1.dae" scale="0.001 0.001 0.001"/>
 				</geometry>
 				<material name="Green">
@@ -47,5 +47,5 @@
 				<origin xyz="0 0 0" rpy="0 0 0"/>
 				<geometry>
-					<mesh filename="package://staubli/meshes/rx60l/visual/rx60bl_hb2.stl" scale="0.001 0.001 0.001"/>
+					<mesh filename="package://staubli_description/meshes/rx60l/visual/rx60bl_hb2.stl" scale="0.001 0.001 0.001"/>
 				</geometry>
 				<material name="White">
@@ -56,5 +56,5 @@
 				<origin xyz="0 0 0" rpy="0 0 0"/>
 				<geometry>
-					<mesh filename="package://staubli/meshes/rx60l/visual/rx60bl_hb2.stl" scale="0.001 0.001 0.001"/>
+					<mesh filename="package://staubli_description/meshes/rx60l/visual/rx60bl_hb2.stl" scale="0.001 0.001 0.001"/>
 				</geometry>
 				<material name="Blue">
@@ -67,5 +67,5 @@
 				<origin xyz="0 0 0" rpy="0 0 0"/>
 				<geometry>
-					<mesh filename="package://staubli/meshes/rx60l/visual/rx60bl_hb3.dae" scale="0.001 0.001 0.001"/>
+					<mesh filename="package://staubli_description/meshes/rx60l/visual/rx60bl_hb3.dae" scale="0.001 0.001 0.001"/>
 				</geometry>
 				<material name="Red">
@@ -76,5 +76,5 @@
 				<origin xyz="0 0 0" rpy="0 0 0"/>
 				<geometry>
-					<mesh filename="package://staubli/meshes/rx60l/visual/rx60bl_hb3.dae" scale="0.001 0.001 0.001"/>
+					<mesh filename="package://staubli_description/meshes/rx60l/visual/rx60bl_hb3.dae" scale="0.001 0.001 0.001"/>
 				</geometry>
 				<material name="Blue">
@@ -87,5 +87,5 @@
 				<origin xyz="0 0 0" rpy="0 0 0"/>
 				<geometry>
-					<mesh filename="package://staubli/meshes/rx60l/visual/rx60bl_hb4.dae" scale="0.001 0.001 0.001"/>
+					<mesh filename="package://staubli_description/meshes/rx60l/visual/rx60bl_hb4.dae" scale="0.001 0.001 0.001"/>
 				</geometry>
 				<material name="Blue">
@@ -96,5 +96,5 @@
 				<origin xyz="0 0 0" rpy="0 0 0"/>
 				<geometry>
-					<mesh filename="package://staubli/meshes/rx60l/visual/rx60bl_hb4.dae" scale="0.001 0.001 0.001"/>
+					<mesh filename="package://staubli_description/meshes/rx60l/visual/rx60bl_hb4.dae" scale="0.001 0.001 0.001"/>
 				</geometry>
 				<material name="Blue">
@@ -107,5 +107,5 @@
 				<origin xyz="0 0 0" rpy="0 0 0"/>
 				<geometry>
-					<mesh filename="package://staubli/meshes/rx60l/visual/rx60bl_hb5.dae" scale="0.001 0.001 0.001"/>
+					<mesh filename="package://staubli_description/meshes/rx60l/visual/rx60bl_hb5.dae" scale="0.001 0.001 0.001"/>
 				</geometry>
 				<material name="Blue">
@@ -127,5 +127,5 @@
 				<origin xyz="0 0 0" rpy="0 0 0"/>
 				<geometry>
-					<mesh filename="package://staubli/meshes/rx60l/visual/rx60bl_hb6.dae" scale="0.001 0.001 0.001"/>
+					<mesh filename="package://staubli_description/meshes/rx60l/visual/rx60bl_hb6.dae" scale="0.001 0.001 0.001"/>
 				</geometry>
 				<material name="Gray">
@@ -136,5 +136,5 @@
 				<origin xyz="0 0 0" rpy="0 0 0"/>
 				<geometry>
-					<mesh filename="package://staubli/meshes/rx60l/visual/rx60bl_hb6.dae" scale="0.001 0.001 0.001"/>
+					<mesh filename="package://staubli_description/meshes/rx60l/visual/rx60bl_hb6.dae" scale="0.001 0.001 0.001"/>
 				</geometry>
 				<material name="Gray">

File: urdf/tx60l.xacro (robot description, xacro)
@@ -1,5 +1,5 @@
 <?xml version="1.0" ?>
 <robot name="staubli_rx60l" xmlns:xacro="http://ros.org/wiki/xacro">
-	<xacro:include filename="$(find staubli)/urdf/tx60l_macro.xacro"/>
+	<xacro:include filename="$(find staubli_description)/urdf/tx60l_macro.xacro"/>
 	<xacro:staubli_rx60l prefix=""/>
 </robot>

File: urdf/tx60l_macro.xacro (robot description, xacro)
@@ -8,5 +8,5 @@
 				<origin xyz="0 0 0" rpy="0 0 0"/>
 				<geometry>
-					<mesh filename="package://staubli/meshes/tx60l/collada/1.dae" scale="${scale}"/>
+					<mesh filename="package://staubli_description/meshes/tx60l/collada/1.dae" scale="${scale}"/>
 				</geometry>
 				<material name="Yellow">
@@ -17,5 +17,5 @@
 				<origin xyz="0 0 0" rpy="0 0 0"/>
 				<geometry>
-					<mesh filename="package://staubli/meshes/tx60l/collada/1.dae" scale="${scale}"/>
+					<mesh filename="package://staubli_description/meshes/tx60l/collada/1.dae" scale="${scale}"/>
 				</geometry>
 				<material name="Blue">
@@ -28,5 +28,5 @@
 				<origin xyz="0 0 0" rpy="0 0 0"/>
 				<geometry>
-					<mesh filename="package://staubli/meshes/tx60l/collada/2.dae" scale="${scale}"/>
+					<mesh filename="package://staubli_description/meshes/tx60l/collada/2.dae" scale="${scale}"/>
 				</geometry>
 				<material name="Yellow">
@@ -37,5 +37,5 @@
 				<origin xyz="0 0 0" rpy="0 0 0"/>
 				<geometry>
-					<mesh filename="package://staubli/meshes/tx60l/collada/2.dae" scale="${scale}"/>
+					<mesh filename="package://staubli_description/meshes/tx60l/collada/2.dae" scale="${scale}"/>
 				</geometry>
 				<material name="Green">
@@ -48,5 +48,5 @@
 				<origin xyz="-0.4 0 0" rpy="0 0 0"/>
 				<geometry>
-					<mesh filename="package://staubli/meshes/tx60l/collada/3.dae" scale="${scale}"/>
+					<mesh filename="package://staubli_description/meshes/tx60l/collada/3.dae" scale="${scale}"/>
 				</geometry>
 				<material name="White">
@@ -57,5 +57,5 @@
 				<origin xyz="-0.4 0 0" rpy="0 0 0"/>
 				<geometry>
-					<mesh filename="package://staubli/meshes/tx60l/collada/3.dae" scale="${scale}"/>
+					<mesh filename="package://staubli_description/meshes/tx60l/collada/3.dae" scale="${scale}"/>
 				</geometry>
 				<material name="Blue">
@@ -68,5 +68,5 @@
 				<origin xyz="0 0 0" rpy="0 0 0"/>
 				<geometry>
-					<mesh filename="package://staubli/meshes/tx60l/collada/4.dae" scale="${scale}"/>
+					<mesh filename="package://staubli_description/meshes/tx60l/collada/4.dae" scale="${scale}"/>
 				</geometry>
 				<material name="Red">
@@ -77,5 +77,5 @@
 				<origin xyz="0 0 0" rpy="0 0 0"/>
 				<geometry>
-					<mesh filename="package://staubli/meshes/tx60l/collada/4.dae" scale="${scale}"/>
+					<mesh filename="package://staubli_description/meshes/tx60l/collada/4.dae" scale="${scale}"/>
 				</geometry>
 				<material name="Blue">
@@ -88,5 +88,5 @@
 				<origin xyz="0 0 0" rpy="0 0 0"/>
 				<geometry>
-					<mesh filename="package://staubli/meshes/tx60l/collada/5.dae" scale="${scale}"/>
+					<mesh filename="package://staubli_description/meshes/tx60l/collada/5.dae" scale="${scale}"/>
 				</geometry>
 				<material name="Blue">
@@ -97,5 +97,5 @@
 				<origin xyz="0 0 0" rpy="0 0 0"/>
 				<geometry>
-					<mesh filename="package://staubli/meshes/tx60l/collada/5.dae" scale="${scale}"/>
+					<mesh filename="package://staubli_description/meshes/tx60l/collada/5.dae" scale="${scale}"/>
 				</geometry>
 				<material name="Blue">
@@ -108,5 +108,5 @@
 				<origin xyz="0 0 0" rpy="0 0 0"/>
 				<geometry>
-					<mesh filename="package://staubli/meshes/tx60l/collada/6.dae" scale="${scale}"/>
+					<mesh filename="package://staubli_description/meshes/tx60l/collada/6.dae" scale="${scale}"/>
 				</geometry>
 				<material name="Blue">
@@ -117,5 +117,5 @@
 				<origin xyz="0 0 0" rpy="0 0 0"/>
 				<geometry>
-					<mesh filename="package://staubli/meshes/tx60l/collada/6.dae" scale="${scale}"/>
+					<mesh filename="package://staubli_description/meshes/tx60l/collada/6.dae" scale="${scale}"/>
 				</geometry>
 				<material name="Blue">
@@ -128,5 +128,5 @@
 				<origin xyz="0 0 0" rpy="0 0 0"/>
 				<geometry>
-					<mesh filename="package://staubli/meshes/tx60l/collada/7.dae" scale="${scale}"/>
+					<mesh filename="package://staubli_description/meshes/tx60l/collada/7.dae" scale="${scale}"/>
 				</geometry>
 				<material name="Gray">
@@ -137,5 +137,5 @@
 				<origin xyz="0 0 0" rpy="0 0 0"/>
 				<geometry>
-					<mesh filename="package://staubli/meshes/tx60l/collada/7.dae" scale="${scale}"/>
+					<mesh filename="package://staubli_description/meshes/tx60l/collada/7.dae" scale="${scale}"/>
 				</geometry>
 				<material name="Gray">
